File: launch.kicad_pcb (KiCad board)
At the start: 4 copper layers, 299 x 127 mm, 347 parts, among them J0 12401598E4#2A, J1 AVR-ISP-6, J2 1003-002-01100, J3 1003-002-01100, J4 12401598E4#2A, J5 12401598E4#2A, U0 USBLC6-2SC6, U1 ATmega32U4-MU, U10 AP22811AW5-7, U11 PTN5110DHQ, U12 PTN5110THQ, U13 PTN5110THQ, U14 SN74LVC1G08DCKR, U15 CBTL02043BBQ,115, U16 AP22811AW5-7‎, U17 TLV62585PDRLR, U18 LP5907MFX-3.3, U19 SN74LVC1G08DCKR, U2 USB7206, U20 AP22811AW5-7, U21 USBLC6-2SC6, U22 AP22811AW5-7, U23 AP22811AW5-7, U3 CBTL02043BBQ,115, U4 TLV62585PDRLR, U5 USBLC6-2SC6, U6 CBTL02043BBQ,115, U7 USBLC6-2SC6, U8 USBLC6-2SC6, U9 AP22811AW5-7, X1 ECS-3225MV-250-BN-TR, Y0 16Mhz

Commit message: fix min solder mask width this was causing no mask to be present between a few QFN ground pads and leads
Other:
- rule pad_to_mask_clearance: 0.051 -> 0.05
- rule solder_mask_min_width: 0.25 -> 0.075

Commit message: use PE2 for LED instead of key matrix closes #7 @jackpot51, note some column lines were swapped for layout purposes
Parts:
- R14: value 12 k -> 9.1 k
- moved R4 1.21 mm to (282.9, 90.4), turned to 90 degrees
Connections:
- R4 pad 1: COLA -> LED
- U1 pad 1: LED -> COLI
- U1 pad 25: COLI -> COLH
- U1 pad 26: COLH -> COLG
- U1 pad 27: COLG -> COLA
- U1 pad 33: COLA -> LED
Routing:
- net COLI: track 226.4 -> 218.2 mm
- net LED: track 15.0 -> 18.8 mm, vias 2 -> 1
- net COLA: track 371.1 -> 374.4 mm
- net GND: track 343.5 -> 342.4 mm
- net COLG: track 258.0 -> 259.0 mm
- net COLF: track 282.2 -> 281.4 mm
- net COLE: track 294.2 -> 293.5 mm
- net COLD: track 312.2 -> 311.5 mm
- net COLC: track 330.7 -> 330.1 mm

Commit message: fix Kailh_socket footprint Put the SMD pads on the top layer so it appears in the correct pick and place file Flipped the entire footprint, then all instances of it on the PCB. closes #1
Parts:
- SWA0, SWA1, SWA2, SWA3, SWA4, SWA5, SWB0, SWB1, SWB2, SWB3, SWB4, SWB5, SWC0, SWC1, SWC2, SWC3, SWC4, SWC5, SWD0, SWD1, SWD2, SWD3, SWD4, SWD5, SWE0, SWE1, SWE2, SWE3, SWE4, SWE5, SWF0, SWF1, SWF2, SWF3, SWF4, SWF5, SWG0, SWG1, SWG2, SWG3, SWG4, SWG5, SWH0, SWH1, SWH2, SWH3, SWH4, SWH5, SWI0, SWI1, SWI2, SWI3, SWI4, SWI5, SWJ0, SWJ1, SWJ2, SWJ3, SWJ4, SWJ5, SWK0, SWK1, SWK2, SWK3, SWK4, SWK5, SWL0, SWL1, SWL2, SWL3, SWL4, SWL5, SWM0, SWM1, SWM2, SWM3, SWM4, SWM5, SWN0, SWN1, SWN2, SWN3, SWN4, SWN5: moved to B.Cu
Other:
- board text added: "6 GND 4 MOSI 2 VCC 3.3 V"
- board text removed: "6 GND 4 MISO 2 VCC 3.3 V"

Commit message: reduce paste mask opening size by 25 μm on USB7206 Issue #5
Routing:
- net GND: vias 287 -> 271
