File: pcb/launch.kicad_pcb (KiCad board)
At the start: 4 copper layers, 299 x 127 mm, 369 parts, among them J0 12401598E4#2A, J1 DNP, J2 1003-002-01100, J3 1003-002-01100, J4 12401598E4#2A, J5 12401598E4#2A, U0 USBLC6-2SC6, U1 ATmega32U4-MU, U10 AP22811AW5-7, U11 PTN5110DHQ, U12 PTN5110THQ, U13 PTN5110THQ, U14 SN74LVC1G08DCKR, U15 CBTL02043ABQ,115, U16 AP22811AW5-7‎, U17 TLV62585PDRLR, U18 LP5907MFX-3.3, U19 SN74LVC1G08DCKR, U2 USB7206, U20 AP22811AW5-7, U21 USBLC6-2SC6, U22 AP22811AW5-7, U23 AP22811AW5-7, U3 CBTL02043ABQ,115, U4 TLV62585PDRLR, U5 USBLC6-2SC6, U6 CBTL02043ABQ,115, U7 USBLC6-2SC6, U8 USBLC6-2SC6, U9 AP22811AW5-7, X1 ECS-3225MV-250-BN-TR, Y0 ECS-160-18-23G-JGN-TR

Commit message: revert accidental removal of System76 logo
Parts:
- added G***: LOGO, Logo:System76, B.Cu at (17.4, -6.55)

Commit message: add logo to schematic, link with PCB
Parts:
- LOGO1: renamed from G***; value LOGO -> System76Logo
Changed lines of the file:
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@@
   (module Logo:System76 (layer B.Cu)
     (at 17.45 -6.55 180)
-    (fp_text reference G*** (at 0 0 180) (layer B.SilkS) hide
+    (fp_text reference LOGO1 (at 0 0 180) (layer B.SilkS) hide
       (effects (font (size 1.524 1.524) (thickness 0.3)) (justify mirror))
     )
-    (fp_text value LOGO (at 0.75 0 180) (layer B.SilkS) hide
+    (fp_text value System76Logo (at 0.75 0 180) (layer B.SilkS) hide
       (effects (font (size 1.524 1.524) (thickness 0.3)) (justify mirror))
     )

Commit message: Ensure correct VBUS capacitor part number
Parts:
- C44, C45, C46, C47: value EEEFK0J151SR -> APXF6R3ARA151ME40G
Changed lines of the file:
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@@
       (effects (font (size 1 1) (thickness 0.15)) (justify mirror))
     )
-    (fp_text value EEEFK0J151SR (at 0 -3.7) (layer B.Fab) hide
+    (fp_text value APXF6R3ARA151ME40G (at 0 -3.7) (layer B.Fab) hide
       (effects (font (size 1 1) (thickness 0.15)) (justify mirror))
     )
@@
       (effects (font (size 1 1) (thickness 0.15)) (justify mirror))
     )
-    (fp_text value EEEFK0J151SR (at 0 -3.7) (layer B.Fab) hide
+    (fp_text value APXF6R3ARA151ME40G (at 0 -3.7) (layer B.Fab) hide
       (effects (font (size 1 1) (thickness 0.15)) (justify mirror))
     )
@@
       (effects (font (size 1 1) (thickness 0.15)) (justify mirror))
     )
-    (fp_text value EEEFK0J151SR (at 0 -3.7) (layer B.Fab) hide
+    (fp_text value APXF6R3ARA151ME40G (at 0 -3.7) (layer B.Fab) hide
       (effects (font (size 1 1) (thickness 0.15)) (justify mirror))
     )
@@
       (effects (font (size 1 1) (thickness 0.15)) (justify mirror))
     )
-    (fp_text value EEEFK0J151SR (at 0 -3.7) (layer B.Fab) hide
+    (fp_text value APXF6R3ARA151ME40G (at 0 -3.7) (layer B.Fab) hide
       (effects (font (size 1 1) (thickness 0.15)) (justify mirror))
     )
