File: pcb/power.kicad_sch (KiCad schematic)
At the start: 26 parts, among them U16 AP22811AW5-7‎, U18 LP5907MFX-3.3, U4 AP3441LSHE-7B

Commit message: work in progress toward 2.0
Parts:
- removed U4: AP3441LSHE-7B, launch:W-DFN2020-8_Type_C, symbol launch:AP3441LSHE-7B
- added U17, U4: MT3410LB, kicad_pcb:SOT-23-5, symbol launch:MT3410LB
Connections:
- net FB1V1: now also U4.5 (FB)
- net FB3V6: now also U17.5 (FB)
- net GND: now also U17.2 (GND), U4.2 (GND)
- net SW1V1: now also U4.3 (SW)
- net SW3V6: now also U17.3 (SW)
- net VCC: now also U17.1 (EN), U17.4 (VIN), U4.1 (EN), U4.4 (VIN)
