File: pcb/USB.kicad_sch (KiCad schematic)
At the start: 101 parts, among them J0 12401598E4#2A, J2 1003-002-01100, J3 1003-002-01100, J4 12401598E4#2A, J5 12401598E4#2A, U0 USBLC6-2SC6, U10 AP22811AW5-7, U11 PTN5110NHQZ, U12 PTN5110NHQZ, U13 PTN5110NHQZ, U14 SN74LVC1G08DCKR, U15 CBTL02043ABQ,115, U19 SN74LVC1G08DCKR, U2 USB7206T/KDX, U20 AP22811AW5-7, U21 USBLC6-2SC6, U23 AP22811AW5-7, U3 CBTL02043ABQ,115, U5 USBLC6-2SC6, U6 CBTL02043ABQ,115, U7 USBLC6-2SC6, U8 USBLC6-2SC6, U9 AP22811AW5-7, X1 ECS-3225MV-250-BN-TR

Commit message: add 2nd SWD connector, BOM edits, export
Parts:
- X1: value ECS-3225MV-250-BN-TR -> ECS-3225MV-250-BN-TR
Changed lines of the file:
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@@
     (title "Launch")
     (date "2023-02-03")
-    (rev "pre 3.0")
+    (rev "3.0")
     (company "System76")
   )
@@
       (effects (font (size 1.27 1.27)) (justify left))
     )
-    (property "Value" " ECS-3225MV-250-BN-TR " (at 147.32 200.66 0)
+    (property "Value" "ECS-3225MV-250-BN-TR " (at 147.32 200.66 0)
       (effects (font (size 1.27 1.27)) (justify left))
     )
