File: pcb-lite/launch-lite.kicad_sch (KiCad schematic)
At the start: 209 parts, among them J0 TYPE-C-31-M-12, J1 DNP, J6 DNP, U0 USBLC6-2SC6, U1 AT90USB646-MUR, Y0 ECS-160-18-23G-JGN-TR

Commit message: launch lite finalization set version to 1.0 copper to NPTH clearance increased to 0.5 mm reroute a few traces move entire PCB by 50, 50 mm to get off of sheet frame
Other:
- title: Launch -> Launch Lite
