File: pcb-lite/power.kicad_sch (KiCad schematic)
At the start: 16 parts, among them U16 AP22811AW5-7‎, U4 M3406-ADJ

Commit message: launch lite finalization set version to 1.0 copper to NPTH clearance increased to 0.5 mm reroute a few traces move entire PCB by 50, 50 mm to get off of sheet frame
Other:
- title: Launch -> Launch Lite
Changed lines of the file:
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@@
-(kicad_sch (version 20210621) (generator eeschema)
+(kicad_sch (version 20211123) (generator eeschema)
   (paper "A4")
   (title_block
-    (title "Launch")
+    (title "Launch Lite")
     (date "2021-09-13")
-    (rev "1.x")
+    (rev "1.0")
     (company "System76")
   )
-  (junction (at 163.83 144.78) (diameter 0) (color 0 0 0 0))
-  (junction (at 114.3 105.41) (diameter 0) (color 0 0 0 0))
-  (junction (at 163.83 135.89) (diameter 0) (color 0 0 0 0))
-  (junction (at 100.33 135.89) (diameter 0) (color 0 0 0 0))
-  (junction (at 114.3 135.89) (diameter 0) (color 0 0 0 0))
-  (junction (at 176.53 135.89) (diameter 0) (color 0 0 0 0))
-  (junction (at 180.34 135.89) (diameter 0) (color 0 0 0 0))
-  (junction (at 167.64 135.89) (diameter 0) (color 0 0 0 0))
-  (junction (at 189.23 135.89) (diameter 0) (color 0 0 0 0))
+  (junction (at 163.83 135.89) (diameter 0) (color 0 0 0 0)
+  )
+  (junction (at 167.64 135.89) (diameter 0) (color 0 0 0 0)
+  )
+  (junction (at 176.53 135.89) (diameter 0) (color 0 0 0 0)
+  )
+  (junction (at 189.23 135.89) (diameter 0) (color 0 0 0 0)
+  )
+  (junction (at 114.3 135.89) (diameter 0) (color 0 0 0 0)
+  )
+  (junction (at 163.83 144.78) (diameter 0) (color 0 0 0 0)
+  )
+  (junction (at 180.34 135.89) (diameter 0) (color 0 0 0 0)
+  )
+  (junction (at 100.33 135.89) (diameter 0) (color 0 0 0 0)
+  )
+  (junction (at 114.3 105.41) (diameter 0) (color 0 0 0 0)
+  )
   (no_connect (at 133.35 110.49))
   (polyline (pts (xy 111.76 127) (xy 172.72 127))
