File: pcb-tenkey/launch-tenkey.kicad_pcb (KiCad board)
At the start: 2 copper layers, 76 x 112 mm, 64 parts, among them J7 FH12-16S-0.5SH(55)

Commit message: version pins, finalize routing FFC connector changed to 20 pin USB hub reset pull down via stitching route remaining nets and cleanup
Parts:
- added C10: 100 nF, Capacitor_SMD:C_0603_1608Metric, B.Cu at (69.0, 115.8)
- added C2: 100 nF, Capacitor_SMD:C_0603_1608Metric, B.Cu at (69.0, 40.4)
- added C3: 100 nF, Capacitor_SMD:C_0603_1608Metric, B.Cu at (88.0, 87.4)
- added C4: 100 nF, Capacitor_SMD:C_0603_1608Metric, B.Cu at (31.0, 40.4)
- added C5: 100 nF, Capacitor_SMD:C_0603_1608Metric, B.Cu at (88.0, 59.0)
- added C6: 100 nF, Capacitor_SMD:C_0603_1608Metric, B.Cu at (50.0, 78.4)
- added C7: 100 nF, Capacitor_SMD:C_0603_1608Metric, B.Cu at (50.0, 97.0)
- added C8: 100 nF, Capacitor_SMD:C_0603_1608Metric, B.Cu at (69.0, 135.0)
- added C9: 100 nF, Capacitor_SMD:C_0603_1608Metric, B.Cu at (31.0, 116.0)
- C1: value 1 uF -> 100 nF
- J7: value FH12-16S-0.5SH(55) -> AFC07-S20FCC-00; footprint Connector_FFC-FPC:Hirose_FH12-16S-0.5SH_1x16-1MP_P0.50mm_Horizontal -> launch:AFC07-S20FCC-00
Connections:
- J7 pad 10: /ROW11 -> /COLM
- J7 pad 11: /ROW10 -> GND
- J7 pad 12: /ROW9 -> /ROW11
- J7 pad 13: /ROW8 -> /ROW10
- J7 pad 14: /ROW7 -> /ROW9
- J7 pad 15: /ROW6 -> GND
- J7 pad 16: GND -> /ROW8
- J7 pad 2: +3V6 -> GND
- J7 pad 4: /LEDI -> +3V6
- J7 pad 5: /COLD -> /LEDI
- J7 pad 6: /COLE -> /COLD
- J7 pad 7: /COLF -> GND
- J7 pad 8: /COLM -> /COLE
- J7 pad 9: GND -> /COLF
Routing:
- net +3V6: track 456.9 -> 335.4 mm, vias 4 -> 11
- net Net-(D46-Pad2): track 21.0 -> 13.6 mm
- net Net-(LA4-Pad1): track 32.9 -> 28.8 mm
- net Net-(D47-Pad1): track 20.8 -> 16.8 mm
- net GND: track 20.0 -> 23.6 mm, vias 53 -> 141
- net Net-(LD1-Pad1): track 34.3 -> 36.0 mm
- net /ROW8: track 70.6 -> 72.1 mm
- net /ROW11: track 34.2 -> 35.3 mm
- net Net-(D10-Pad1): track 21.8 -> 22.8 mm
- net Net-(LA2-Pad1): track 26.7 -> 25.7 mm
- net /COLD: track 8.58 -> 9.55 mm
- net /ROW6: track 115.2 -> 114.7 mm, vias 3 -> 2
- added copper zone on F.Cu, net +3V6
