File: pcb-heavy/launch-heavy.kicad_sch (KiCad schematic)
At the start: 73 parts, among them J7 AFC07-S20FCC-00

Commit message: rename launch-tenkey to launch-heavy
Other:
- title: Launch Ten Key -> Launch Heavy
Changed lines of the file:
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@@
   (paper "A4")
   (title_block
-    (title "Launch Ten Key")
+    (title "Launch Heavy")
     (date "2022-05-19")
     (rev "0.0")

Commit message: set versions
Parts:
- J7: Manufacturer (none) -> Jushou
Changed lines of the file:
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@@
   (title_block
     (title "Launch Heavy")
-    (date "2022-05-19")
-    (rev "0.0")
+    (date "2022-05-23")
+    (rev "1.0")
     (company "System76")
   )
@@
       (effects (font (size 1.27 1.27)) hide)
     )
-    (property "Datasheet" "~" (id 3) (at 44.45 38.1 0)
+    (property "Datasheet" "https://assets.nexperia.com/documents/data-sheet/BAV70_SER.pdf" (id 3) (at 44.45 38.1 0)
       (effects (font (size 1.27 1.27)) hide)
     )
@@
       (effects (font (size 1.27 1.27)) hide)
     )
-    (property "Datasheet" "~" (id 3) (at 44.45 50.8 0)
+    (property "Datasheet" "https://assets.nexperia.com/documents/data-sheet/BAV70_SER.pdf" (id 3) (at 44.45 50.8 0)
       (effects (font (size 1.27 1.27)) hide)
     )
@@
       (effects (font (size 1.27 1.27)) hide)
     )
-    (property "Datasheet" "~" (id 3) (at 44.45 63.5 0)
+    (property "Datasheet" "https://assets.nexperia.com/documents/data-sheet/BAV70_SER.pdf" (id 3) (at 44.45 63.5 0)
       (effects (font (size 1.27 1.27)) hide)
     )
@@
       (effects (font (size 1.27 1.27)) hide)
     )
-    (property "Datasheet" "~" (id 3) (at 44.45 76.2 0)
+    (property "Datasheet" "https://assets.nexperia.com/documents/data-sheet/BAV70_SER.pdf" (id 3) (at 44.45 76.2 0)
       (effects (font (size 1.27 1.27)) hide)
     )
@@
       (effects (font (size 1.27 1.27)) hide)
     )
-    (property "Datasheet" "~" (id 3) (at 44.45 88.9 0)
+    (property "Datasheet" "https://assets.nexperia.com/documents/data-sheet/BAV70_SER.pdf" (id 3) (at 44.45 88.9 0)
       (effects (font (size 1.27 1.27)) hide)
     )
@@
       (effects (font (size 1.27 1.27)) hide)
     )
-    (property "Datasheet" "~" (id 3) (at 44.45 101.6 0)
+    (property "Datasheet" "https://assets.nexperia.com/documents/data-sheet/BAV70_SER.pdf" (id 3) (at 44.45 101.6 0)
       (effects (font (size 1.27 1.27)) hide)
     )
@@
       (effects (font (size 1.27 1.27)) hide)
     )
-    (property "Datasheet" "~" (id 3) (at 82.55 38.1 0)
+    (property "Datasheet" "https://assets.nexperia.com/documents/data-sheet/BAV70_SER.pdf" (id 3) (at 82.55 38.1 0)
       (effects (font (size 1.27 1.27)) hide)
     )
@@
       (effects (font (size 1.27 1.27)) hide)
     )
-    (property "Datasheet" "~" (id 3) (at 82.55 50.8 0)
+    (property "Datasheet" "https://assets.nexperia.com/documents/data-sheet/BAV70_SER.pdf" (id 3) (at 82.55 50.8 0)
       (effects (font (size 1.27 1.27)) hide)
     )
@@
       (effects (font (size 1.27 1.27)) hide)
     )
-    (property "Datasheet" "~" (id 3) (at 82.55 63.5 0)
+    (property "Datasheet" "https://assets.nexperia.com/documents/data-sheet/BAV70_SER.pdf" (id 3) (at 82.55 63.5 0)
       (effects (font (size 1.27 1.27)) hide)
     )
@@
       (effects (font (size 1.27 1.27)) hide)
     )
-    (property "Datasheet" "~" (id 3) (at 82.55 76.2 0)
+    (property "Datasheet" "https://assets.nexperia.com/documents/data-sheet/BAV70_SER.pdf" (id 3) (at 82.55 76.2 0)
       (effects (font (size 1.27 1.27)) hide)
     )
@@
       (effects (font (size 1.27 1.27)) hide)
     )
-    (property "Datasheet" "~" (id 3) (at 82.55 88.9 0)
+    (property "Datasheet" "https://assets.nexperia.com/documents/data-sheet/BAV70_SER.pdf" (id 3) (at 82.55 88.9 0)
       (effects (font (size 1.27 1.27)) hide)
     )
@@
       (effects (font (size 1.27 1.27)) hide)
     )
+    (property "Manufacturer" "Jushou" (id 4) (at 219.71 101.6 0)
+      (effects (font (size 1.27 1.27)) hide)
+    )
