File: pcb-iso/launch-iso.kicad_sch (KiCad schematic)
At the start: 244 parts, among them J1 DNP, J6 DNP, J7 AFC07-S20FCC-00, U1 AT90USB646-MUR, Y0 ECS-160-18-23G-JGN-TR

Commit message: clean up routing, schematic title block
Other:
- title: Launch -> Launch ISO
Changed lines of the file:
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@@
   (paper "A3")
   (title_block
-    (title "Launch")
-    (date "2022-05-24")
+    (title "Launch ISO")
+    (date "2022-08-16")
     (rev "2.0")
     (company "System76")
