File: pcb-iso/power.kicad_sch (KiCad schematic)
At the start: 27 parts, among them U16 AP22811AW5-7‎, U17 MT3410LB, U18 LP5907MFX-3.3, U4 MT3410LB

Commit message: clean up routing, schematic title block
Other:
- title: Launch -> Launch ISO
Changed lines of the file:
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@@
   (paper "A4")
   (title_block
-    (title "Launch")
-    (date "2022-05-24")
+    (title "Launch ISO")
+    (date "2022-08-16")
     (rev "2.0")
     (company "System76")
